Commit message: Rviz now works

File: src/qube_description/urdf/qube.macro.xacro (robot description, xacro)
@@ -1,4 +1,4 @@
 <?xml version = "1.0"?>
-<robot xmls:xacro = "https://wwww.ros.org/wiki/xacro">
+<robot xmlns:xacro = "https://wwww.ros.org/wiki/xacro">
     <xacro:macro name = "qube">
         <xacro:property name = "baseSize" value = "0.1" />
@@ -9,5 +9,5 @@
             <visual>
                 <geometry>
-                    <box size = "${baseSize} ${baseSize} ${baseSize}">
+					<box size = "${baseSize} ${baseSize} ${baseSize}"/>
                 </geometry>
                 <material name =  "black">
@@ -38,5 +38,5 @@
             </visual>
         </link>
-        <-- Koblinger (Joints) -->
+        <!-- Koblinger (Joints) -->
         <joint name = "indicatorJoint" type = "fixed">
             <parent link = "disk"/>
@@ -44,3 +44,9 @@
             <origin xyz = "0 ${diskRadius} 0"/>
         </joint>
+        <joint name = "diskJoint" type = "fixed">
+            <parent link = "baseLink"/>
+            <child link = "disk"/>
+            <origin xyz = "0 ${diskRadius} 0"/>
+        </joint>
+	</xacro:macro>
 </robot>

Commit message: Oppgave 1 done

File: src/qube_description/urdf/qube.macro.xacro (robot description, xacro)
@@ -3,5 +3,5 @@
     <xacro:macro name = "qube">
         <xacro:property name = "baseSize" value = "0.1" />
-        <xacro:property name = "diskRadius" value = "0.05" />
+		<xacro:property name = "diskRadius" value = "${baseSize / 4}" />
         <xacro:property name = "diskHeight" value = "0.01" />
         <!--Svart boks -->
@@ -31,5 +31,5 @@
             <visual>
                 <geometry>
-                    <box size = "0.01 0.32 0.002"/>
+					<box size = "${diskHeight * 0.2} ${diskRadius} ${diskHeight*1.1}"/>
                 </geometry>
                 <material name = "white">
@@ -39,13 +39,13 @@
         </link>
         <!-- Koblinger (Joints) -->
+        <joint name = "diskJoint" type = "fixed">
+            <parent link = "baseLink"/>
+            <child link = "disk"/>
+			<origin xyz = "0 0 ${baseSize / 2}"/>
+        </joint>
         <joint name = "indicatorJoint" type = "fixed">
             <parent link = "disk"/>
             <child link = "indicator"/>
-            <origin xyz = "0 ${diskRadius} 0"/>
-        </joint>
-        <joint name = "diskJoint" type = "fixed">
-            <parent link = "baseLink"/>
-            <child link = "disk"/>
-            <origin xyz = "0 ${diskRadius} 0"/>
+			<origin xyz = "0 ${diskRadius / 2} 0"/>
         </joint>
 	</xacro:macro>
