Commit message: Not working, but maybe progress on task 3

File: src/qube_bringup/urdf/controlled_qube.urdf.xacro (robot description, xacro)
@@ -2,6 +2,6 @@
 <robot xmlns:xacro = "https://www.ros.org/wiki/xacro">
     <!-- Argumenter -->
-    <xacro:arg name = "baudRate" default = "115200">
-    <xacro:arg name = "device" default = "/dev/ttyACM0">
+	<xacro:arg name = "baud_rate" default = "115200"/>
+	<xacro:arg name = "device" default = "/dev/ttyACM0"/>
     <xacro:arg name = "simulation" default = "false"/>
     <!-- Inkluder beskrivelse av qube -->
@@ -14,5 +14,5 @@
         name = "qube_driver"
         prefix = ""
-        baudRate = "$(arg baudRate)"
+        baud_rate = "$(arg baud_rate)"
         device = "$(arg device)"
         simulation = "$(arg simulation)"/>

File: src/qube_description/urdf/qube.urdf.xacro (robot description, xacro)
@@ -1,7 +1,7 @@
 <?xml version = "1.0"?>
 <robot name="qube" xmlns:xacro = "https://wwww.ros.org/wiki/xacro">
-<xacro:include filename="$(find qube_description)/urdf/qube.macro.xacro" />
-<link name = "world"/>
-<xacro:qube/>
+	<xacro:include filename="$(find qube_description)/urdf/qube.macro.xacro" />
+	<link name = "world"/>
+	<xacro:qube/>
 	<joint name = "worldJoint" type = "fixed">
 		<parent link = "world"/>

Commit message: Bringup seems to be working

File: src/qube_bringup/urdf/controlled_qube.urdf.xacro (robot description, xacro)
@@ -1,8 +1,8 @@
 <?xml version = "1.0"?>
-<robot xmlns:xacro = "https://www.ros.org/wiki/xacro">
+<robot name="qube" xmlns:xacro = "https://www.ros.org/wiki/xacro">
     <!-- Argumenter -->
 	<xacro:arg name = "baud_rate" default = "115200"/>
 	<xacro:arg name = "device" default = "/dev/ttyACM0"/>
-    <xacro:arg name = "simulation" default = "false"/>
+    <xacro:arg name = "simulation" default = "true"/>
     <!-- Inkluder beskrivelse av qube -->
     <xacro:include filename = "$(find qube_description)/urdf/qube.macro.xacro"/>
@@ -17,4 +17,5 @@
         device = "$(arg device)"
         simulation = "$(arg simulation)"/>
+	<link name = "world"/>
     <!-- World link -->
     <joint name = "base_to_world" type = "fixed">

File: src/qube_description/urdf/qube.macro.xacro (robot description, xacro)
@@ -39,5 +39,5 @@
         </link>
         <!-- Koblinger (Joints) -->
-        <joint name = "diskJoint" type = "fixed">
+        <joint name = "motor_joint" type = "continuous">
             <parent link = "baseLink"/>
             <child link = "disk"/>

Commit message: Everything works in simulation at least

File: src/qube_bringup/urdf/controlled_qube.urdf.xacro (robot description, xacro)
@@ -4,5 +4,5 @@
 	<xacro:arg name = "baud_rate" default = "115200"/>
 	<xacro:arg name = "device" default = "/dev/ttyACM0"/>
-    <xacro:arg name = "simulation" default = "true"/>
+    <xacro:arg name = "simulation" default = "false"/>
     <!-- Inkluder beskrivelse av qube -->
     <xacro:include filename = "$(find qube_description)/urdf/qube.macro.xacro"/>

File: src/qube_description/urdf/qube.macro.xacro (robot description, xacro)
@@ -42,4 +42,5 @@
             <parent link = "baseLink"/>
             <child link = "disk"/>
+			<axis xyz = "0 0 1"/>
 			<origin xyz = "0 0 ${baseSize / 2}"/>
         </joint>

Commit message: Pid tuned

File: src/qube_bringup/urdf/controlled_qube.urdf.xacro (robot description, xacro)
@@ -4,5 +4,5 @@
 	<xacro:arg name = "baud_rate" default = "115200"/>
 	<xacro:arg name = "device" default = "/dev/ttyACM0"/>
-    <xacro:arg name = "simulation" default = "false"/>
+    <xacro:arg name = "simulation" default = "true"/>
     <!-- Inkluder beskrivelse av qube -->
     <xacro:include filename = "$(find qube_description)/urdf/qube.macro.xacro"/>

File: src/qube_description/urdf/qube.macro.xacro (robot description, xacro)
@@ -5,5 +5,5 @@
 		<xacro:property name = "diskRadius" value = "${baseSize / 4}" />
         <xacro:property name = "diskHeight" value = "0.01" />
-        <!--Svart boks -->
+        <!-- Svart boks -->
         <link name = "baseLink">
             <visual>
@@ -16,5 +16,5 @@
             </visual>
         </link>
-        <!--Rød disk -->
+        <!-- Rød disk -->
         <link name = "disk">
             <visual>
@@ -27,5 +27,5 @@
             </visual>
         </link>
-        <!--Hvit viser(indikator) -->
+        <!-- Indikator -->
         <link name = "indicator">
             <visual>
@@ -38,9 +38,10 @@
             </visual>
         </link>
-        <!-- Koblinger (Joints) -->
+        <!-- Joints -->
         <joint name = "motor_joint" type = "continuous">
             <parent link = "baseLink"/>
             <child link = "disk"/>
-			<axis xyz = "0 0 1"/>
+			<!-- Invert rotation to follow real one correctly -->
+			<axis xyz = "0 0 -1"/>
 			<origin xyz = "0 0 ${baseSize / 2}"/>
         </joint>
